File: GameHma.kicad_pcb (KiCad board)
At the start: 2 copper layers, 95 x 70 mm, 22 parts, among them J1 Screw_Terminal_01x02, J2 Motor_Terminal_01x04, J3 Motor_Terminal_01x04, J4 Motor_Terminal_01x04, J5 Motor_Terminal_01x04, J6 Conn_01x03, U1 ESP32-DEVKIT-V1, U2 A4988 Stepper Driver Module, U3 A4988 Stepper Driver Module, U4 A4988 Stepper Driver Module, U5 A4988 Stepper Driver Module, U6 SRT_MP1584EN

Commit message: KiCad update: 2026-01-06 14:31:30
Routing:
- net +V_{DD}: track 314.3 -> 314.8 mm
Changed lines of the file:
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@@
-	)
-	(segment
-		(start 33.6 35.75)
-		(end 22.939575 35.75)
-		(width 1.016)
-		(layer "B.Cu")
-		(net 26)
 	)
 	(segment
@@
 	)
 	(segment
-		(start 20.25 38.439575)
-		(end 20.25 43.75)
-		(width 1.016)
-		(layer "B.Cu")
-		(net 26)
-	)
-	(segment
 		(start 98.8139 81.5639)
 		(end 97.2785 81.5639)
@@
 		(start 41.922973 49.74715)
 		(end 40.25 48.074177)
+		(width 1.016)
+		(layer "B.Cu")
+		(net 26)
+	)
+	(segment
+		(start 33.6 35.75)
+		(end 22 35.75)
 		(width 1.016)
 		(layer "B.Cu")
@@
 	)
 	(segment
+		(start 20.25 37.5)
+		(end 20.25 43.75)
+		(width 1.016)
+		(layer "B.Cu")
+		(net 26)
+	)
+	(segment
 		(start 93.15 56.9)
 		(end 95.15285 54.89715)
@@
 	)
 	(segment
-		(start 86.5 59.525)
-		(end 86.4875 59.5125)
+		(start 22 35.75)
+		(end 20.25 37.5)
 		(width 1.016)
 		(layer "B.Cu")
@@
 	)
 	(segment
-		(start 22.939575 35.75)
-		(end 20.25 38.439575)
+		(start 86.5 59.525)
+		(end 86.4875 59.5125)
 		(width 1.016)
 		(layer "B.Cu")
